Commit message: adding camera

File: description/robot.urdf.xacro (robot description, xacro)
@@ -3,3 +3,5 @@
     <xacro:include filename="robot_core.xacro" />
     <xacro:include filename="robot_control.xacro" />
+    <xacro:include filename="lidar.xacro" />
+    <xacro:include filename="camera.xacro" />
 </robot>

File: description/robot_control.xacro (robot description, xacro)
@@ -2,4 +2,6 @@
 <robot xmlns:xacro="http://www.ros.org/xacro" name="robot">
     <gazebo>
+        <!-- The plugin listens to the /cmd_vel topic for velocity commands to control the robot. -->
+        <!-- The plugin publishes to the /odom topic to provide odometry data (e.g., position and velocity of the robot). -->
         <plugin name="diff_drive" filename="libgazebo_ros_diff_drive.so">
             <!-- Wheel information -->

File: description/robot_core.xacro (robot description, xacro)
@@ -16,4 +16,7 @@
     <material name="black">
         <color rgba="0 0 0 1"/>
+    </material>
+    <material name="red">
+        <color rgba="1 0 0 1"/>
     </material>
     <!-- BASE LINK -->
