Commit message: new changes

File: description/camera.xacro (robot description, xacro)
@@ -21,5 +21,6 @@
         <origin xyz="0 0 0 " rpy="${-pi/2} 0 ${-pi/2}"/>
     </joint>
-     <link name="camera_link_optical"></link>
+    <link name="camera_link_optical">
+    </link>
     <gazebo reference="camera_link">
         <material>Gazebo/Red</material>
@@ -40,5 +41,6 @@
                 </clip>
             </camera>
-            <plugin name="camera_controller" filename="libgazebo_ros_camera_sensor.so">
+            <!-- Maybe change this -->
+            <plugin name="camera_controller" filename="libgazebo_ros_camera.so">
                 <frame_name>camera_link_optical</frame_name>
             </plugin>

File: description/lidar.xacro (robot description, xacro)
@@ -1,10 +1,10 @@
 <?xml version="1.0"?>
 <robot xmlns:xacro="http://www.ros.org/wiki/xacro"  name="robot">
-    <joint name="lidar_joint" type="fixed">
+    <joint name="laser_joint" type="fixed">
         <parent link="chassis" />
-        <child link="lidar"/>
+        <child link="laser_frame"/>
         <origin xyz="0.1 0 0.175" rpy="0 0 0"/>
     </joint>
-    <link name="lidar">
+    <link name="laser_frame">
         <visual>
             <geometry>
@@ -32,4 +32,5 @@
                     <horizontal>
                         <samples>360</samples>
+                        <resolution>1</resolution>
                         <min_angle>-3.14</min_angle>
                         <max_angle>3.14</max_angle>
@@ -39,4 +40,5 @@
                     <min>0.3</min>
                     <max>12</max>
+                    <resolution>0.1</resolution>
                 </range>
             </ray>
@@ -46,5 +48,5 @@
                 </ros>
                 <output_type>sensor_msgs/LaserScan</output_type>
-                <frame_name>lidar</frame_name>
+                <frame_name>laser_frame</frame_name>
             </plugin>
         </sensor>
